File: pcb/soundspy-node.kicad_pcb (KiCad board)
At the start: 2 copper layers, 30 x 68 mm, 9 parts, among them U1_L ESP32_L, U1_R ESP32_R

Commit message: PCB: fix mic connector to correct 2x3 2.54mm footprint, remove all traces
- Replace wrong 1x5 1.27mm header with correct 2x3 2.54mm layout
- Pin layout: GND/VDD/SD (top row), LR/WS/SCK (bottom row)
- Row separation 7.62mm, column pitch 2.54mm (from barafael/inmp441-breakout-kicad)
- Pad drill 0.762mm, pad size 1.524mm
- Sound port hole corrected to 3mm
- Added I2S_LR net (L/R select pin, ties to GND for left channel)
- Removed all crossing traces — ready for routing in KiCad
Parts:
- J_MIC: value ICS-43434 -> INMP441-Breakout; footprint Connector_PinHeader_1.27mm:PinHeader_1x05_P1.27mm_Vertical -> Connector_PinHeader_2.54mm:PinHeader_2x03_P2.54mm_Vertical
- SOUND_PORT: footprint MountingHole:MountingHole_1.5mm -> MountingHole:MountingHole_3.2mm
- moved J_MIC 2.73 mm to (15.0, 5.50)
- moved C1 2.69 mm to (22.0, 5.50)
- moved SOUND_PORT 2.00 mm to (15.0, 5.50)
Connections:
- J_MIC pad 1: 3V3 -> GND
- J_MIC pad 2: GND -> 3V3
- J_MIC pad 3: I2S_WS -> I2S_SD
- J_MIC pad 4: I2S_SD -> I2S_LR
- J_MIC pad 5: I2S_SCK -> I2S_WS
Routing:
- net I2S_SD: track 83.6 -> 0.00 mm
- net I2S_WS: track 40.5 -> 0.00 mm
- net GND: track 31.9 -> 0.00 mm
- net 3V3: track 22.7 -> 0.00 mm
Other:
- board text added: "SoundSpy Node v1.1"
- board text removed: "SoundSpy Node v1.0"
Changed lines of the file:
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@@
     (title "SoundSpy Node Carrier")
     (date "2026-07-30")
-    (rev "1.0")
-    (comment 1 "ESP32 38-pin DevKit + ICS-43434 carrier board")
+    (rev "1.1")
+    (comment 1 "ESP32 38-pin DevKit + INMP441/ICS-43434 circular breakout carrier")
     (comment 2 "USB-C notch at bottom for case passthrough")
-    (comment 3 "Mic on standoffs, port facing front")
+    (comment 3 "Mic module: 14mm dia, 2x3 header 2.54mm col / 7.62mm row pitch")
   )
   (layers
@@
   (net 4 "I2S_SD")
   (net 5 "I2S_SCK")
-  (gr_line (start 0 0)   (end 30 0)  (layer "Edge.Cuts") (width 0.15))
-  (gr_line (start 30 0)  (end 30 68) (layer "Edge.Cuts") (width 0.15))
-  (gr_line (start 0 68)  (end 0 0)   (layer "Edge.Cuts") (width 0.15))
-  (gr_line (start 0 68)   (end 9.5 68)  (layer "Edge.Cuts") (width 0.15))
-  (gr_line (start 9.5 68) (end 9.5 64)  (layer "Edge.Cuts") (width 0.15))
-  (gr_line (start 9.5 64) (end 20.5 64) (layer "Edge.Cuts") (width 0.15))
-  (gr_line (start 20.5 64)(end 20.5 68) (layer "Edge.Cuts") (width 0.15))
-  (gr_line (start 20.5 68)(end 30 68)   (layer "Edge.Cuts") (width 0.15))
+  (net 6 "I2S_LR")
+  (gr_line (start 0 0)    (end 30 0)   (layer "Edge.Cuts") (width 0.15))
+  (gr_line (start 30 0)   (end 30 68)  (layer "Edge.Cuts") (width 0.15))
+  (gr_line (start 0 68)   (end 0 0)    (layer "Edge.Cuts") (width 0.15))
+  (gr_line (start 0 68)   (end 9.5 68) (layer "Edge.Cuts") (width 0.15))
+  (gr_line (start 9.5 68) (end 9.5 64) (layer "Edge.Cuts") (width 0.15))
+  (gr_line (start 9.5 64) (end 20.5 64)(layer "Edge.Cuts") (width 0.15))
+  (gr_line (start 20.5 64)(end 20.5 68)(layer "Edge.Cuts") (width 0.15))
+  (gr_line (start 20.5 68)(end 30 68)  (layer "Edge.Cuts") (width 0.15))
   (footprint "MountingHole:MountingHole_2.2mm_M2" (at 3 3) (layer "F.Cu")
     (uuid "mh000001")
@@
     (pad "" np_thru_hole circle (at 0 0) (size 2.2 2.2) (drill 2.2) (layers "*.Cu" "*.Mask") (uuid "mhp000004"))
   )
-  (footprint "Connector_PinHeader_1.27mm:PinHeader_1x05_P1.27mm_Vertical" (at 12.46 4.5 0) (layer "F.Cu")
-    (fp_text reference "J_MIC" (at 2.54 -1.5) (layer "F.SilkS") (effects (font (size 0.7 0.7) (thickness 0.1))))
-    (fp_text value "ICS-43434" (at 2.54 1.5) (layer "F.Fab") (effects (font (size 0.7 0.7) (thickness 0.1))))
-    (pad "1" thru_hole rect   (at 0 0)     (size 1.5 1.5) (drill 0.8) (layers "*.Cu" "*.Mask") (net 1 "3V3"))
-    (pad "2" thru_hole circle (at 1.27 0)  (size 1.5 1.5) (drill 0.8) (layers "*.Cu" "*.Mask") (net 2 "GND"))
-    (pad "3" thru_hole circle (at 2.54 0)  (size 1.5 1.5) (drill 0.8) (layers "*.Cu" "*.Mask") (net 3 "I2S_WS"))
-    (pad "4" thru_hole circle (at 3.81 0)  (size 1.5 1.5) (drill 0.8) (layers "*.Cu" "*.Mask") (net 4 "I2S_SD"))
-    (pad "5" thru_hole circle (at 5.08 0)  (size 1.5 1.5) (drill 0.8) (layers "*.Cu" "*.Mask") (net 5 "I2S_SCK"))
+  (footprint "Connector_PinHeader_2.54mm:PinHeader_2x03_P2.54mm_Vertical" (at 15 5.5 0) (layer "F.Cu")
+    (fp_text reference "J_MIC" (at 0 -3.0) (layer "F.SilkS") (effects (font (size 0.8 0.8) (thickness 0.12))))
+    (fp_text value "INMP441-Breakout" (at 0 3.5) (layer "F.Fab") (effects (font (size 0.7 0.7) (thickness 0.1))))
+    (fp_text user "GND" (at -3.0 -3.81 0) (layer "F.SilkS") (effects (font (size 0.6 0.6) (thickness 0.09))))
+    (fp_text user "VDD" (at 0 -3.81 0)    (layer "F.SilkS") (effects (font (size 0.6 0.6) (thickness 0.09))))
+    (fp_text user "SD"  (at 3.0 -3.81 0)  (layer "F.SilkS") (effects (font (size 0.6 0.6) (thickness 0.09))))
+    (fp_text user "LR"  (at -3.0 3.81 0)  (layer "F.SilkS") (effects (font (size 0.6 0.6) (thickness 0.09))))
+    (fp_text user "WS"  (at 0 3.81 0)     (layer "F.SilkS") (effects (font (size 0.6 0.6) (thickness 0.09))))
+    (fp_text user "SCK" (at 3.0 3.81 0)   (layer "F.SilkS") (effects (font (size 0.6 0.6) (thickness 0.09))))
+    (pad "1" thru_hole rect   (at -2.54 -3.81) (size 1.524 1.524) (drill 0.762) (layers "*.Cu" "*.Mask") (net 2 "GND"))
+    (pad "2" thru_hole circle (at 0     -3.81) (size 1.524 1.524) (drill 0.762) (layers "*.Cu" "*.Mask") (net 1 "3V3"))
+    (pad "3" thru_hole circle (at 2.54  -3.81) (size 1.524 1.524) (drill 0.762) (layers "*.Cu" "*.Mask") (net 4 "I2S_SD"))
+    (pad "4" thru_hole circle (at -2.54  3.81) (size 1.524 1.524) (drill 0.762) (layers "*.Cu" "*.Mask") (net 6 "I2S_LR"))
+    (pad "5" thru_hole circle (at 0      3.81) (size 1.524 1.524) (drill 0.762) (layers "*.Cu" "*.Mask") (net 3 "I2S_WS"))
+    (pad "6" thru_hole circle (at 2.54   3.81) (size 1.524 1.524) (drill 0.762) (layers "*.Cu" "*.Mask") (net 5 "I2S_SCK"))
   )
-  (footprint "MountingHole:MountingHole_1.5mm" (at 15 7.5) (layer "F.Cu")
-    (fp_text reference "SOUND_PORT" (at 0 -2) (layer "F.SilkS") (effects (font (size 0.5 0.5) (thickness 0.08))))
-    (pad "" np_thru_hole circle (at 0 0) (size 1.5 1.5) (drill 1.5) (layers "*.Cu" "*.Mask"))
+  (footprint "MountingHole:MountingHole_3.2mm" (at 15 5.5) (layer "F.Cu")
+    (fp_text reference "SOUND_PORT" (at 0 -2.5) (layer "F.SilkS") (effects (font (size 0.5 0.5) (thickness 0.08))))
+    (pad "" np_thru_hole circle (at 0 0) (size 3.0 3.0) (drill 3.0) (layers "*.Cu" "*.Mask"))
   )
-  (footprint "Capacitor_SMD:C_0402_1005Metric" (at 19.5 4.5 0) (layer "F.Cu")
+  (footprint "Capacitor_SMD:C_0402_1005Metric" (at 22 5.5 0) (layer "F.Cu")
     (fp_text reference "C1" (at 0 -0.9) (layer "F.SilkS") (effects (font (size 0.6 0.6) (thickness 0.1))))
     (fp_text value "100nF" (at 0 0.9) (layer "F.Fab") (effects (font (size 0.6 0.6) (thickness 0.1))))
@@
     (pad "19" thru_hole circle (at 0 45.72)  (size 1.7 1.7) (drill 1.0) (layers "*.Cu" "*.Mask") (net 0 "")     (uuid "espr000019"))
   )
-  (segment (start 27.7 12.0) (end 27.7 10.0)  (width 0.3) (layer "F.Cu") (net 1) (uuid "tr000001"))
-  (segment (start 27.7 10.0) (end 19.02 10.0) (width 0.3) (layer "F.Cu") (net 1) (uuid "tr000002"))
-  (segment (start 19.02 10.0)(end 19.02 4.5)  (width 0.3) (layer "F.Cu") (net 1) (uuid "tr000003"))
-  (segment (start 18.98 4.5) (end 12.46 4.5)  (width 0.3) (layer "F.Cu") (net 1) (uuid "tr000004"))
-  (segment (start 2.3 12.0)  (end 2.3 10.5)   (width 0.3) (layer "F.Cu") (net 2) (uuid "tr000005"))
-  (segment (start 2.3 10.5)  (end 7.0 10.5)   (width 0.3) (layer "F.Cu") (net 2) (uuid "tr000006"))
-  (segment (start 7.0 10.5)  (end 7.0 4.5)    (width 0.3) (layer "F.Cu") (net 2) (uuid "tr000007"))
-  (segment (start 7.0 4.5)   (end 13.73 4.5)  (width 0.3) (layer "F.Cu") (net 2) (uuid "tr000008"))
-  (segment (start 7.0 4.5)   (end 19.98 4.5)  (width 0.3) (layer "F.Cu") (net 2) (uuid "tr000009"))
-  (segment (start 2.3 32.32) (end 5.5 32.32)  (width 0.25) (layer "F.Cu") (net 3) (uuid "tr000010"))
-  (segment (start 5.5 32.32) (end 5.5 6.0)    (width 0.25) (layer "F.Cu") (net 3) (uuid "tr000011"))
-  (segment (start 5.5 6.0)   (end 15.0 6.0)   (width 0.25) (layer "F.Cu") (net 3) (uuid "tr000012"))
-  (segment (start 15.0 6.0)  (end 15.0 4.5)   (width 0.25) (layer "F.Cu") (net 3) (uuid "tr000013"))
-  (segment (start 2.3 29.78) (end 6.5 29.78)  (width 0.25) (layer "F.Cu") (net 4) (uuid "tr000014"))
-  (segment (start 6.5 29.78) (end 6.5 6.5)    (width 0.25) (layer "F.Cu") (net 4) (uuid "tr000015"))
-  (segment (start 6.5 6.5)   (end 16.27 6.5)  (width 0.25) (layer "F.Cu") (net 4) (uuid "tr000016"))
-  (segment (start 16.27 6.5) (end 16.27 4.5)  (width 0.25) (layer "F.Cu") (net 4) (uuid "tr000017"))
-  (segment (start 2.3 34.86) (end 6.5 34.86)  (width 0.25) (layer "F.Cu") (net 4) (uuid "tr000018"))
-  (segment (start 6.5 34.86) (end 6.5 7.0)    (width 0.25) (layer "F.Cu") (net 4) (uuid "tr000019"))
-  (segment (start 6.5 7.0)   (end 16.27 7.0)  (width 0.25) (layer "F.Cu") (net 4) (uuid "tr000020"))
-  (segment (start 16.27 7.0) (end 16.27 4.5)  (width 0.25) (layer "F.Cu") (net 4) (uuid "tr000021"))
-  (gr_text "SoundSpy Node v1.0" (at 15 61.0) (layer "F.SilkS")
+  (gr_text "SoundSpy Node v1.1" (at 15 61.0) (layer "F.SilkS")
     (effects (font (size 0.8 0.8) (thickness 0.12)))
   )
-  (gr_text "MIC" (at 15 2.5) (layer "F.SilkS")
+  (gr_text "MIC" (at 15 1.5) (layer "F.SilkS")
     (effects (font (size 0.7 0.7) (thickness 0.1)))
   )
